File: cad/rotary_board.kicad_pcb (KiCad board)
At the start: 2 copper layers, 6.7 x 15.2 mm, 1 part, among them J1 USB_C_Receptacle

Commit message: add files
Parts:
- removed J1: USB_C_Receptacle, usb-type-c:CX70M-24P1
- added C1: 22p, Capacitor_SMD:CP_Elec_3x5.3, F.Cu at (628.6, 216.7)
- added C2: 22p, Capacitor_SMD:CP_Elec_3x5.3, F.Cu at (628.6, 221.5)
- added D1: D, Diode_SMD:D_SOD-123, B.Cu at (7.14, 54.8)
- added D10: D, Diode_SMD:D_SOD-123, B.Cu at (33.3, 131.0)
- added D100: WS2812B, LED_SMD:LED_WS2812B_PLCC4_5.0x5.0mm_P3.2mm, F.Cu at (331.0, 250.0)
- added D101: WS2812B, LED_SMD:LED_WS2812B_PLCC4_5.0x5.0mm_P3.2mm, F.Cu at (321.5, 250.0)
- added D11: D, Diode_SMD:D_SOD-123, B.Cu at (45.2, 54.8)
- added D12: D, Diode_SMD:D_SOD-123, B.Cu at (54.8, 73.8)
- added D13: D, Diode_SMD:D_SOD-123, B.Cu at (59.5, 92.9)
- added D14: D, Diode_SMD:D_SOD-123, B.Cu at (69.1, 111.9)
- added D15: D, Diode_SMD:D_SOD-123, B.Cu at (57.1, 131.0)
- added D16: D, Diode_SMD:D_SOD-123, B.Cu at (64.3, 54.8)
- added D17: D, Diode_SMD:D_SOD-123, B.Cu at (73.8, 73.8)
- added D18: D, Diode_SMD:D_SOD-123, B.Cu at (78.6, 92.9)
- added D19: D, Diode_SMD:D_SOD-123, B.Cu at (88.1, 111.9)
- added D2: D, Diode_SMD:D_SOD-123, B.Cu at (11.9, 73.8)
- added D20: D, Diode_SMD:D_SOD-123, B.Cu at (83.3, 54.8)
- added D21: D, Diode_SMD:D_SOD-123, B.Cu at (92.9, 73.8)
- added D22: D, Diode_SMD:D_SOD-123, B.Cu at (97.6, 92.9)
- added D23: D, Diode_SMD:D_SOD-123, B.Cu at (107.2, 111.9)
- added D24: D, Diode_SMD:D_SOD-123, B.Cu at (102.4, 54.8)
- added D25: D, Diode_SMD:D_SOD-123, B.Cu at (111.9, 73.8)
- added D26: D, Diode_SMD:D_SOD-123, B.Cu at (116.7, 92.9)
- added D27: D, Diode_SMD:D_SOD-123, B.Cu at (126.2, 111.9)
- added D28: D, Diode_SMD:D_SOD-123, B.Cu at (131.0, 131.0)
- added D29: D, Diode_SMD:D_SOD-123, B.Cu at (121.4, 54.8)
- added D3: D, Diode_SMD:D_SOD-123, B.Cu at (14.3, 92.9)
- added D30: D, Diode_SMD:D_SOD-123, B.Cu at (131.0, 73.8)
- added D31: D, Diode_SMD:D_SOD-123, B.Cu at (135.7, 92.9)
- added D32: D, Diode_SMD:D_SOD-123, B.Cu at (145.3, 111.9)
- added D33: D, Diode_SMD:D_SOD-123, B.Cu at (140.5, 54.8)
- added D34: D, Diode_SMD:D_SOD-123, B.Cu at (150.0, 73.8)
- added D35: D, Diode_SMD:D_SOD-123, B.Cu at (154.8, 92.9)
- added D36: D, Diode_SMD:D_SOD-123, B.Cu at (164.3, 111.9)
- added D37: D, Diode_SMD:D_SOD-123, B.Cu at (159.5, 54.8)
- added D38: D, Diode_SMD:D_SOD-123, B.Cu at (169.1, 73.8)
- added D39: D, Diode_SMD:D_SOD-123, B.Cu at (173.8, 92.9)
- added D4: D, Diode_SMD:D_SOD-123, B.Cu at (19.1, 111.9)
- added D40: D, Diode_SMD:D_SOD-123, B.Cu at (183.4, 111.9)
- added D41: D, Diode_SMD:D_SOD-123, B.Cu at (204.8, 131.0)
- added D42: D, Diode_SMD:D_SOD-123, B.Cu at (178.6, 54.8)
- added D43: D, Diode_SMD:D_SOD-123, B.Cu at (188.1, 73.8)
- added D44: D, Diode_SMD:D_SOD-123, B.Cu at (192.9, 92.9)
- added D45: D, Diode_SMD:D_SOD-123, B.Cu at (202.4, 111.9)
- added D46: D, Diode_SMD:D_SOD-123, B.Cu at (226.2, 131.0)
- added D47: D, Diode_SMD:D_SOD-123, B.Cu at (197.6, 54.8)
- added D48: D, Diode_SMD:D_SOD-123, B.Cu at (207.2, 73.8)
- added D49: D, Diode_SMD:D_SOD-123, B.Cu at (211.9, 92.9)
- added D5: D, Diode_SMD:D_SOD-123, B.Cu at (9.53, 131.0)
- added D50: D, Diode_SMD:D_SOD-123, B.Cu at (221.5, 111.9)
- added D51: D, Diode_SMD:D_SOD-123, B.Cu at (247.7, 131.0)
- added D52: D, Diode_SMD:D_SOD-123, B.Cu at (216.7, 54.8)
- added D53: D, Diode_SMD:D_SOD-123, B.Cu at (226.2, 73.8)
- added D54: D, Diode_SMD:D_SOD-123, B.Cu at (231.0, 92.9)
- added D55: D, Diode_SMD:D_SOD-123, B.Cu at (257.2, 111.9)
- added D56: D, Diode_SMD:D_SOD-123, B.Cu at (269.1, 73.8)
- added D57: D, Diode_SMD:D_SOD-123, B.Cu at (235.7, 54.8)
- added D58: D, Diode_SMD:D_SOD-123, B.Cu at (245.3, 73.8)
- added D59: D, Diode_SMD:D_SOD-123, B.Cu at (261.9, 92.9)
- added D6: D, Diode_SMD:D_SOD-123, B.Cu at (26.2, 54.8)
- added D60: D, Diode_SMD:D_SOD-123, B.Cu at (264.3, 54.8)
- added D61: D, Diode_SMD:D_SOD-123, B.Cu at (271.5, 131.0)
- added D62: D, Diode_SMD:D_SOD-123, B.Cu at (354.8, 76.2)
- added D63: D, Diode_SMD:D_SOD-123, B.Cu at (321.5, 152.4)
- added D64: D, Diode_SMD:D_SOD-123, B.Cu at (321.5, 171.4)
- added D65: D, Diode_SMD:D_SOD-123, B.Cu at (321.5, 190.5)
- added D66: D, Diode_SMD:D_SOD-123, B.Cu at (369.1, 76.2)
- added D67: D, Diode_SMD:D_SOD-123, B.Cu at (345.3, 152.4)
- added D68: D, Diode_SMD:D_SOD-123, B.Cu at (345.3, 171.4)
- added D69: D, Diode_SMD:D_SOD-123, B.Cu at (345.3, 190.5)
- added D7: D, Diode_SMD:D_SOD-123, B.Cu at (35.7, 73.8)
- added D70: WS2812B, LED_SMD:LED_WS2812B_PLCC4_5.0x5.0mm_P3.2mm, F.Cu at (388.1, 261.9)
- added D71: WS2812B, LED_SMD:LED_WS2812B_PLCC4_5.0x5.0mm_P3.2mm, F.Cu at (378.6, 261.9)
- added D72: WS2812B, LED_SMD:LED_WS2812B_PLCC4_5.0x5.0mm_P3.2mm, F.Cu at (369.1, 261.9)
- added D73: WS2812B, LED_SMD:LED_WS2812B_PLCC4_5.0x5.0mm_P3.2mm, F.Cu at (388.1, 238.1)
- added D74: WS2812B, LED_SMD:LED_WS2812B_PLCC4_5.0x5.0mm_P3.2mm, F.Cu at (378.6, 238.1)
- added D75: WS2812B, LED_SMD:LED_WS2812B_PLCC4_5.0x5.0mm_P3.2mm, F.Cu at (369.1, 238.1)
- added D76: WS2812B, LED_SMD:LED_WS2812B_PLCC4_5.0x5.0mm_P3.2mm, F.Cu at (359.6, 261.9)
- added D77: WS2812B, LED_SMD:LED_WS2812B_PLCC4_5.0x5.0mm_P3.2mm, F.Cu at (350.0, 261.9)
- added D78: WS2812B, LED_SMD:LED_WS2812B_PLCC4_5.0x5.0mm_P3.2mm, F.Cu at (340.5, 261.9)
- added D79: WS2812B, LED_SMD:LED_WS2812B_PLCC4_5.0x5.0mm_P3.2mm, F.Cu at (359.6, 238.1)
- added D8: D, Diode_SMD:D_SOD-123, B.Cu at (40.5, 92.9)
- added D80: WS2812B, LED_SMD:LED_WS2812B_PLCC4_5.0x5.0mm_P3.2mm, F.Cu at (350.0, 238.1)
- added D81: WS2812B, LED_SMD:LED_WS2812B_PLCC4_5.0x5.0mm_P3.2mm, F.Cu at (340.5, 238.1)
- added D82: WS2812B, LED_SMD:LED_WS2812B_PLCC4_5.0x5.0mm_P3.2mm, F.Cu at (331.0, 261.9)
- added D83: WS2812B, LED_SMD:LED_WS2812B_PLCC4_5.0x5.0mm_P3.2mm, F.Cu at (321.5, 261.9)
- added D84: WS2812B, LED_SMD:LED_WS2812B_PLCC4_5.0x5.0mm_P3.2mm, F.Cu at (331.0, 238.1)
- added D85: WS2812B, LED_SMD:LED_WS2812B_PLCC4_5.0x5.0mm_P3.2mm, F.Cu at (321.5, 238.1)
- added D86: WS2812B, LED_SMD:LED_WS2812B_PLCC4_5.0x5.0mm_P3.2mm, F.Cu at (362.7, 86.4)
- added D87: WS2812B, LED_SMD:LED_WS2812B_PLCC4_5.0x5.0mm_P3.2mm, F.Cu at (351.1, 81.5)
- added D88: WS2812B, LED_SMD:LED_WS2812B_PLCC4_5.0x5.0mm_P3.2mm, F.Cu at (346.2, 69.8)
- added D89: WS2812B, LED_SMD:LED_WS2812B_PLCC4_5.0x5.0mm_P3.2mm, F.Cu at (388.1, 250.0)
- added D9: D, Diode_SMD:D_SOD-123, B.Cu at (50.0, 111.9)
- added D90: WS2812B, LED_SMD:LED_WS2812B_PLCC4_5.0x5.0mm_P3.2mm, F.Cu at (378.6, 250.0)
- added D91: WS2812B, LED_SMD:LED_WS2812B_PLCC4_5.0x5.0mm_P3.2mm, F.Cu at (369.1, 250.0)
- added D92: WS2812B, LED_SMD:LED_WS2812B_PLCC4_5.0x5.0mm_P3.2mm, F.Cu at (351.1, 58.2)
- added D93: WS2812B, LED_SMD:LED_WS2812B_PLCC4_5.0x5.0mm_P3.2mm, F.Cu at (362.7, 53.3)
- added D94: WS2812B, LED_SMD:LED_WS2812B_PLCC4_5.0x5.0mm_P3.2mm, F.Cu at (374.4, 58.2)
- added D95: WS2812B, LED_SMD:LED_WS2812B_PLCC4_5.0x5.0mm_P3.2mm, F.Cu at (359.6, 250.0)
- added D96: WS2812B, LED_SMD:LED_WS2812B_PLCC4_5.0x5.0mm_P3.2mm, F.Cu at (350.0, 250.0)
- added D97: WS2812B, LED_SMD:LED_WS2812B_PLCC4_5.0x5.0mm_P3.2mm, F.Cu at (340.5, 250.0)
- added D98: WS2812B, LED_SMD:LED_WS2812B_PLCC4_5.0x5.0mm_P3.2mm, F.Cu at (379.3, 69.8)
- added D99: WS2812B, LED_SMD:LED_WS2812B_PLCC4_5.0x5.0mm_P3.2mm, F.Cu at (374.4, 81.5)
- added SW1: tilde, Button_Switch_Keyboard:SW_Cherry_MX_1.00u_PCB, F.Cu at (12.1, 44.9)
- added SW10: l_windows, Button_Switch_Keyboard:SW_Cherry_MX_1.25u_PCB, F.Cu at (38.3, 121.1)
- added SW11: two, Button_Switch_Keyboard:SW_Cherry_MX_1.00u_PCB, F.Cu at (50.2, 44.9)
- added SW12: w, Button_Switch_Keyboard:SW_Cherry_MX_1.00u_PCB, F.Cu at (59.7, 64.0)
- added SW13: s, Button_Switch_Keyboard:SW_Cherry_MX_1.00u_PCB, F.Cu at (64.5, 83.0)
- added SW14: x, Button_Switch_Keyboard:SW_Cherry_MX_1.00u_PCB, F.Cu at (74.0, 102.1)
- added SW15: l_alt, Button_Switch_Keyboard:SW_Cherry_MX_1.25u_PCB, F.Cu at (62.1, 121.1)
- added SW16: three, Button_Switch_Keyboard:SW_Cherry_MX_1.00u_PCB, F.Cu at (69.2, 44.9)
- added SW17: e, Button_Switch_Keyboard:SW_Cherry_MX_1.00u_PCB, F.Cu at (78.7, 64.0)
- added SW18: d, Button_Switch_Keyboard:SW_Cherry_MX_1.00u_PCB, F.Cu at (83.5, 83.0)
- added SW19: c, Button_Switch_Keyboard:SW_Cherry_MX_1.00u_PCB, F.Cu at (93.0, 102.1)
- added SW2: tab, Button_Switch_Keyboard:SW_Cherry_MX_1.50u_PCB, F.Cu at (16.8, 64.0)
- added SW20: four, Button_Switch_Keyboard:SW_Cherry_MX_1.00u_PCB, F.Cu at (88.3, 44.9)
- added SW21: r, Button_Switch_Keyboard:SW_Cherry_MX_1.00u_PCB, F.Cu at (97.8, 64.0)
- added SW22: f, Button_Switch_Keyboard:SW_Cherry_MX_1.00u_PCB, F.Cu at (102.6, 83.0)
- added SW23: v, Button_Switch_Keyboard:SW_Cherry_MX_1.00u_PCB, F.Cu at (112.1, 102.1)
- added SW24: five, Button_Switch_Keyboard:SW_Cherry_MX_1.00u_PCB, F.Cu at (107.3, 44.9)
- added SW25: t, Button_Switch_Keyboard:SW_Cherry_MX_1.00u_PCB, F.Cu at (116.8, 64.0)
- added SW26: g, Button_Switch_Keyboard:SW_Cherry_MX_1.00u_PCB, F.Cu at (121.6, 83.0)
- added SW27: b, Button_Switch_Keyboard:SW_Cherry_MX_1.00u_PCB, F.Cu at (131.1, 102.1)
- added SW28: space, Button_Switch_Keyboard:SW_Cherry_MX_6.25u_PCB, F.Cu at (135.9, 121.1)
- added SW29: six, Button_Switch_Keyboard:SW_Cherry_MX_1.00u_PCB, F.Cu at (126.4, 44.9)
- added SW3: caps_lock, Button_Switch_Keyboard:SW_Cherry_MX_1.75u_PCB, F.Cu at (19.2, 83.0)
- added SW30: y, Button_Switch_Keyboard:SW_Cherry_MX_1.00u_PCB, F.Cu at (135.9, 64.0)
- added SW31: h, Button_Switch_Keyboard:SW_Cherry_MX_1.00u_PCB, F.Cu at (140.7, 83.0)
- added SW32: n, Button_Switch_Keyboard:SW_Cherry_MX_1.00u_PCB, F.Cu at (150.2, 102.1)
- added SW33: seven, Button_Switch_Keyboard:SW_Cherry_MX_1.00u_PCB, F.Cu at (145.4, 44.9)
- added SW34: u, Button_Switch_Keyboard:SW_Cherry_MX_1.00u_PCB, F.Cu at (154.9, 64.0)
- added SW35: j, Button_Switch_Keyboard:SW_Cherry_MX_1.00u_PCB, F.Cu at (159.7, 83.0)
- added SW36: m, Button_Switch_Keyboard:SW_Cherry_MX_1.00u_PCB, F.Cu at (169.2, 102.1)
- added SW37: eight, Button_Switch_Keyboard:SW_Cherry_MX_1.00u_PCB, F.Cu at (164.5, 44.9)
- added SW38: i, Button_Switch_Keyboard:SW_Cherry_MX_1.00u_PCB, F.Cu at (174.0, 64.0)
- added SW39: k, Button_Switch_Keyboard:SW_Cherry_MX_1.00u_PCB, F.Cu at (178.8, 83.0)
- added SW4: left_shift, Button_Switch_Keyboard:SW_Cherry_MX_2.25u_PCB, F.Cu at (24.0, 102.1)
- added SW40: comma, Button_Switch_Keyboard:SW_Cherry_MX_1.00u_PCB, F.Cu at (188.3, 102.1)
- added SW41: r_alt, Button_Switch_Keyboard:SW_Cherry_MX_1.25u_PCB, F.Cu at (209.7, 121.1)
- added SW42: nine, Button_Switch_Keyboard:SW_Cherry_MX_1.00u_PCB, F.Cu at (183.5, 44.9)
- added SW43: o, Button_Switch_Keyboard:SW_Cherry_MX_1.00u_PCB, F.Cu at (193.0, 64.0)
- added SW44: l, Button_Switch_Keyboard:SW_Cherry_MX_1.00u_PCB, F.Cu at (197.8, 83.0)
- added SW45: period, Button_Switch_Keyboard:SW_Cherry_MX_1.00u_PCB, F.Cu at (207.3, 102.1)
- added SW46: r_windows, Button_Switch_Keyboard:SW_Cherry_MX_1.25u_PCB, F.Cu at (231.1, 121.1)
- added SW47: zero, Button_Switch_Keyboard:SW_Cherry_MX_1.00u_PCB, F.Cu at (202.6, 44.9)
- added SW48: p, Button_Switch_Keyboard:SW_Cherry_MX_1.00u_PCB, F.Cu at (212.1, 64.0)
- added SW49: ;, Button_Switch_Keyboard:SW_Cherry_MX_1.00u_PCB, F.Cu at (216.9, 83.0)
- added SW5: l_ctrl, Button_Switch_Keyboard:SW_Cherry_MX_1.25u_PCB, F.Cu at (14.4, 121.1)
- added SW50: /, Button_Switch_Keyboard:SW_Cherry_MX_1.00u_PCB, F.Cu at (226.4, 102.1)
- added SW51: fn, Button_Switch_Keyboard:SW_Cherry_MX_1.25u_PCB, F.Cu at (252.6, 121.1)
- added SW52: hyphen, Button_Switch_Keyboard:SW_Cherry_MX_1.00u_PCB, F.Cu at (221.6, 44.9)
- added SW53: [, Button_Switch_Keyboard:SW_Cherry_MX_1.00u_PCB, F.Cu at (231.1, 64.0)
- added SW54: ', Button_Switch_Keyboard:SW_Cherry_MX_1.00u_PCB, F.Cu at (235.9, 83.0)
- added SW55: right_shift, Button_Switch_Keyboard:SW_Cherry_MX_2.75u_PCB, F.Cu at (262.1, 102.1)
- added SW56: \, Button_Switch_Keyboard:SW_Cherry_MX_1.50u_PCB, F.Cu at (274.0, 64.0)
- added SW57: equals, Button_Switch_Keyboard:SW_Cherry_MX_1.00u_PCB, F.Cu at (240.7, 44.9)
- added SW58: ], Button_Switch_Keyboard:SW_Cherry_MX_1.00u_PCB, F.Cu at (250.2, 64.0)
- added SW59: enter, Button_Switch_Keyboard:SW_Cherry_MX_2.25u_PCB, F.Cu at (266.9, 83.0)
- added SW6: one, Button_Switch_Keyboard:SW_Cherry_MX_1.00u_PCB, F.Cu at (31.1, 44.9)
- added SW60: backspace, Button_Switch_Keyboard:SW_Cherry_MX_2.00u_PCB, F.Cu at (269.2, 44.9)
- added SW61: r_ctrl, Button_Switch_Keyboard:SW_Cherry_MX_1.25u_PCB, F.Cu at (276.4, 121.1)
- added SW62: R1, Rotary_Encoder:RotaryEncoder_Alps_EC11E-Switch_Vertical_H20mm, F.Cu at (354.8, 66.7)
- added SW63: R2, Rotary_Encoder:RotaryEncoder_Alps_EC11E-Switch_Vertical_H20mm, F.Cu at (326.2, 145.3)
- added SW64: R3, Rotary_Encoder:RotaryEncoder_Alps_EC11E-Switch_Vertical_H20mm, F.Cu at (326.2, 164.3)
- added SW65: R4, Rotary_Encoder:RotaryEncoder_Alps_EC11E-Switch_Vertical_H20mm, F.Cu at (326.2, 183.4)
- added SW7: q, Button_Switch_Keyboard:SW_Cherry_MX_1.00u_PCB, F.Cu at (40.6, 64.0)
- added SW8: a, Button_Switch_Keyboard:SW_Cherry_MX_1.00u_PCB, F.Cu at (45.4, 83.0)
- added SW9: z, Button_Switch_Keyboard:SW_Cherry_MX_1.00u_PCB, F.Cu at (54.9, 102.1)
- added U1: AT90USB1286-A, Package_QFP:TQFP-64_14x14mm_P0.8mm, F.Cu at (610.4, 223.5)
- added X1: XTAL_GND, Crystal:Crystal_AT310_D3.0mm_L10.0mm_Horizontal, F.Cu at (621.1, 215.6)
Other:
- board outline removed
