File: cad/rotary_board.sch (KiCad schematic (older format))
At the start: 4 parts, among them X1 XTAL_GND

Commit message: add files
Parts:
- removed U?: ATMEGA32U4, symbol Component_library:ATMEGA32U4
- added D1, D10, D11, D12, D13, D14, D15, D16, D17, D18, D19, D2, D20, D21, D22, D23, D24, D25, D26, D27, D28, D29, D3, D30, D31, D32, D33, D34, D35, D36, D37, D38, D39, D4, D40, D41, D42, D43, D44, D45, D46, D47, D48, D49, D5, D50, D51, D52, D53, D54, D55, D56, D57, D58, D59, D6, D60, D61, D62, D63, D64, D65, D66, D67, D68, D69, D7, D8, D9: D, Diode_SMD:D_SOD-123, symbol Device:D
- added D100, D101, D70, D71, D72, D73, D74, D75, D76, D77, D78, D79, D80, D81, D82, D83, D84, D85, D86, D87, D88, D89, D90, D91, D92, D93, D94, D95, D96, D97, D98, D99: WS2812B, LED_SMD:LED_WS2812B_PLCC4_5.0x5.0mm_P3.2mm, symbol LED:WS2812B
- added SW1: tilde, Button_Switch_Keyboard:SW_Cherry_MX_1.00u_PCB, symbol Switch:SW_Push
- added SW10: l_windows, Button_Switch_Keyboard:SW_Cherry_MX_1.25u_PCB, symbol Switch:SW_Push
- added SW11: two, Button_Switch_Keyboard:SW_Cherry_MX_1.00u_PCB, symbol Switch:SW_Push
- added SW12: w, Button_Switch_Keyboard:SW_Cherry_MX_1.00u_PCB, symbol Switch:SW_Push
- added SW13: s, Button_Switch_Keyboard:SW_Cherry_MX_1.00u_PCB, symbol Switch:SW_Push
- added SW14: x, Button_Switch_Keyboard:SW_Cherry_MX_1.00u_PCB, symbol Switch:SW_Push
- added SW15: l_alt, Button_Switch_Keyboard:SW_Cherry_MX_1.25u_PCB, symbol Switch:SW_Push
- added SW16: three, Button_Switch_Keyboard:SW_Cherry_MX_1.00u_PCB, symbol Switch:SW_Push
- added SW17: e, Button_Switch_Keyboard:SW_Cherry_MX_1.00u_PCB, symbol Switch:SW_Push
- added SW18: d, Button_Switch_Keyboard:SW_Cherry_MX_1.00u_PCB, symbol Switch:SW_Push
- added SW19: c, Button_Switch_Keyboard:SW_Cherry_MX_1.00u_PCB, symbol Switch:SW_Push
- added SW2: tab, Button_Switch_Keyboard:SW_Cherry_MX_1.50u_PCB, symbol Switch:SW_Push
- added SW20: four, Button_Switch_Keyboard:SW_Cherry_MX_1.00u_PCB, symbol Switch:SW_Push
- added SW21: r, Button_Switch_Keyboard:SW_Cherry_MX_1.00u_PCB, symbol Switch:SW_Push
- added SW22: f, Button_Switch_Keyboard:SW_Cherry_MX_1.00u_PCB, symbol Switch:SW_Push
- added SW23: v, Button_Switch_Keyboard:SW_Cherry_MX_1.00u_PCB, symbol Switch:SW_Push
- added SW24: five, Button_Switch_Keyboard:SW_Cherry_MX_1.00u_PCB, symbol Switch:SW_Push
- added SW25: t, Button_Switch_Keyboard:SW_Cherry_MX_1.00u_PCB, symbol Switch:SW_Push
- added SW26: g, Button_Switch_Keyboard:SW_Cherry_MX_1.00u_PCB, symbol Switch:SW_Push
- added SW27: b, Button_Switch_Keyboard:SW_Cherry_MX_1.00u_PCB, symbol Switch:SW_Push
- added SW28: space, Button_Switch_Keyboard:SW_Cherry_MX_6.25u_PCB, symbol Switch:SW_Push
- added SW29: six, Button_Switch_Keyboard:SW_Cherry_MX_1.00u_PCB, symbol Switch:SW_Push
- added SW3: caps_lock, Button_Switch_Keyboard:SW_Cherry_MX_1.75u_PCB, symbol Switch:SW_Push
- added SW30: y, Button_Switch_Keyboard:SW_Cherry_MX_1.00u_PCB, symbol Switch:SW_Push
- added SW31: h, Button_Switch_Keyboard:SW_Cherry_MX_1.00u_PCB, symbol Switch:SW_Push
- added SW32: n, Button_Switch_Keyboard:SW_Cherry_MX_1.00u_PCB, symbol Switch:SW_Push
- added SW33: seven, Button_Switch_Keyboard:SW_Cherry_MX_1.00u_PCB, symbol Switch:SW_Push
- added SW34: u, Button_Switch_Keyboard:SW_Cherry_MX_1.00u_PCB, symbol Switch:SW_Push
- added SW35: j, Button_Switch_Keyboard:SW_Cherry_MX_1.00u_PCB, symbol Switch:SW_Push
- added SW36: m, Button_Switch_Keyboard:SW_Cherry_MX_1.00u_PCB, symbol Switch:SW_Push
- added SW37: eight, Button_Switch_Keyboard:SW_Cherry_MX_1.00u_PCB, symbol Switch:SW_Push
- added SW38: i, Button_Switch_Keyboard:SW_Cherry_MX_1.00u_PCB, symbol Switch:SW_Push
- added SW39: k, Button_Switch_Keyboard:SW_Cherry_MX_1.00u_PCB, symbol Switch:SW_Push
- added SW4: left_shift, Button_Switch_Keyboard:SW_Cherry_MX_2.25u_PCB, symbol Switch:SW_Push
- added SW40: comma, Button_Switch_Keyboard:SW_Cherry_MX_1.00u_PCB, symbol Switch:SW_Push
- added SW41: r_alt, Button_Switch_Keyboard:SW_Cherry_MX_1.25u_PCB, symbol Switch:SW_Push
- added SW42: nine, Button_Switch_Keyboard:SW_Cherry_MX_1.00u_PCB, symbol Switch:SW_Push
- added SW43: o, Button_Switch_Keyboard:SW_Cherry_MX_1.00u_PCB, symbol Switch:SW_Push
- added SW44: l, Button_Switch_Keyboard:SW_Cherry_MX_1.00u_PCB, symbol Switch:SW_Push
- added SW45: period, Button_Switch_Keyboard:SW_Cherry_MX_1.00u_PCB, symbol Switch:SW_Push
- added SW46: r_windows, Button_Switch_Keyboard:SW_Cherry_MX_1.25u_PCB, symbol Switch:SW_Push
- added SW47: zero, Button_Switch_Keyboard:SW_Cherry_MX_1.00u_PCB, symbol Switch:SW_Push
- added SW48: p, Button_Switch_Keyboard:SW_Cherry_MX_1.00u_PCB, symbol Switch:SW_Push
- added SW49: ;, Button_Switch_Keyboard:SW_Cherry_MX_1.00u_PCB, symbol Switch:SW_Push
- added SW5: l_ctrl, Button_Switch_Keyboard:SW_Cherry_MX_1.25u_PCB, symbol Switch:SW_Push
- added SW50: /, Button_Switch_Keyboard:SW_Cherry_MX_1.00u_PCB, symbol Switch:SW_Push
- added SW51: fn, Button_Switch_Keyboard:SW_Cherry_MX_1.25u_PCB, symbol Switch:SW_Push
- added SW52: hyphen, Button_Switch_Keyboard:SW_Cherry_MX_1.00u_PCB, symbol Switch:SW_Push
- added SW53: [, Button_Switch_Keyboard:SW_Cherry_MX_1.00u_PCB, symbol Switch:SW_Push
- added SW54: ', Button_Switch_Keyboard:SW_Cherry_MX_1.00u_PCB, symbol Switch:SW_Push
- added SW55: right_shift, Button_Switch_Keyboard:SW_Cherry_MX_2.75u_PCB, symbol Switch:SW_Push
- added SW56: \\, Button_Switch_Keyboard:SW_Cherry_MX_1.50u_PCB, symbol Switch:SW_Push
- added SW57: equals, Button_Switch_Keyboard:SW_Cherry_MX_1.00u_PCB, symbol Switch:SW_Push
- added SW58: ], Button_Switch_Keyboard:SW_Cherry_MX_1.00u_PCB, symbol Switch:SW_Push
- added SW59: enter, Button_Switch_Keyboard:SW_Cherry_MX_2.25u_PCB, symbol Switch:SW_Push
- added SW6: one, Button_Switch_Keyboard:SW_Cherry_MX_1.00u_PCB, symbol Switch:SW_Push
- added SW60: backspace, Button_Switch_Keyboard:SW_Cherry_MX_2.00u_PCB, symbol Switch:SW_Push
- added SW61: r_ctrl, Button_Switch_Keyboard:SW_Cherry_MX_1.25u_PCB, symbol Switch:SW_Push
- added SW62: R1, Rotary_Encoder:RotaryEncoder_Alps_EC11E-Switch_Vertical_H20mm, symbol Device:Rotary_Encoder_Switch
- added SW63: R2, Rotary_Encoder:RotaryEncoder_Alps_EC11E-Switch_Vertical_H20mm, symbol Device:Rotary_Encoder_Switch
- added SW64: R3, Rotary_Encoder:RotaryEncoder_Alps_EC11E-Switch_Vertical_H20mm, symbol Device:Rotary_Encoder_Switch
- added SW65: R4, Rotary_Encoder:RotaryEncoder_Alps_EC11E-Switch_Vertical_H20mm, symbol Device:Rotary_Encoder_Switch
- added SW7: q, Button_Switch_Keyboard:SW_Cherry_MX_1.00u_PCB, symbol Switch:SW_Push
- added SW8: a, Button_Switch_Keyboard:SW_Cherry_MX_1.00u_PCB, symbol Switch:SW_Push
- added SW9: z, Button_Switch_Keyboard:SW_Cherry_MX_1.00u_PCB, symbol Switch:SW_Push
- added U1: AT90USB1286-A, Package_QFP:TQFP-64_14x14mm_P0.8mm, symbol mcus:AT90USB1286-A
- C1, C2: footprint (none) -> Capacitor_SMD:CP_Elec_3x5.3
- X1: footprint (none) -> Crystal:Crystal_AT310_D3.0mm_L10.0mm_Horizontal
Connections:
- net at C1.1, X1.1: now also U1.24 (XTAL1)
- net at C2.1, X1.2: now also U1.23 (XTAL2)
- new net: D62.2 (A), SW62.C
- new net: D66.2 (A), SW62.S2
- new net: U1.21 (VCC), U1.52 (VCC)
- new net: D1.2 (A), SW1.2
- new net: D6.2 (A), SW6.2
- new net: D11.2 (A), SW11.2
- new net: D16.2 (A), SW16.2
- new net: D20.2 (A), SW20.2
- new net: D24.2 (A), SW24.2
- new net: D33.2 (A), SW33.2
- new net: D37.2 (A), SW37.2
- new net: D42.2 (A), SW42.2
- new net: D29.2 (A), SW29.2
- new net: D47.2 (A), SW47.2
- new net: D52.2 (A), SW52.2
- new net: D56.2 (A), SW56.2
- new net: D61.2 (A), SW61.2
- new net: D57.2 (A), SW57.2
- new net: D48.2 (A), SW48.2
- new net: D53.2 (A), SW53.2
- new net: D58.2 (A), SW58.2
- new net: D30.2 (A), SW30.2
- new net: D43.2 (A), SW43.2
- new net: D38.2 (A), SW38.2
- new net: D34.2 (A), SW34.2
- new net: D25.2 (A), SW25.2
- new net: D7.2 (A), SW7.2
- new net: D21.2 (A), SW21.2
- new net: D17.2 (A), SW17.2
- new net: D12.2 (A), SW12.2
- new net: D2.2 (A), SW2.2
- new net: D49.2 (A), SW49.2
- new net: D54.2 (A), SW54.2
- new net: D59.2 (A), SW59.2
- new net: D31.2 (A), SW31.2
- new net: D44.2 (A), SW44.2
- new net: D39.2 (A), SW39.2
- new net: D35.2 (A), SW35.2
- new net: D26.2 (A), SW26.2
- new net: D8.2 (A), SW8.2
- new net: D22.2 (A), SW22.2
- new net: D18.2 (A), SW18.2
- new net: D13.2 (A), SW13.2
- new net: D3.2 (A), SW3.2
- new net: D50.2 (A), SW50.2
- new net: D55.2 (A), SW55.2
- new net: D60.2 (A), SW60.2
- new net: D32.2 (A), SW32.2
- new net: D45.2 (A), SW45.2
- new net: D40.2 (A), SW40.2
- new net: D36.2 (A), SW36.2
- new net: D27.2 (A), SW27.2
- new net: D9.2 (A), SW9.2
- new net: D23.2 (A), SW23.2
- new net: D19.2 (A), SW19.2
- new net: D14.2 (A), SW14.2
- new net: D4.2 (A), SW4.2
- new net: D51.2 (A), SW51.2
- new net: D46.2 (A), SW46.2
- new net: D41.2 (A), SW41.2
- new net: D28.2 (A), SW28.2
- new net: D10.2 (A), SW10.2
- new net: D15.2 (A), SW15.2
- new net: D5.2 (A), SW5.2
- new net: D63.2 (A), SW63.C
- new net: D67.2 (A), SW63.S2
- new net: D64.2 (A), SW64.C
- new net: D68.2 (A), SW64.S2
- new net: D65.2 (A), SW65.C
- new net: D69.2 (A), SW65.S2
- new net: D70.2 (DOUT), D71.4 (DIN)
- new net: D71.2 (DOUT), D72.4 (DIN)
- new net: D72.2 (DOUT), D76.4 (DIN)
- new net: D78.2 (DOUT), D82.4 (DIN)
- new net: D77.2 (DOUT), D78.4 (DIN)
- new net: D76.2 (DOUT), D77.4 (DIN)
- new net: D82.2 (DOUT), D83.4 (DIN)
- new net: D83.2 (DOUT), D89.4 (DIN)
- new net: D73.2 (DOUT), D74.4 (DIN)
- new net: D101.2 (DOUT), D73.4 (DIN)
- new net: D74.2 (DOUT), D75.4 (DIN)
- new net: D75.2 (DOUT), D79.4 (DIN)
- new net: D81.2 (DOUT), D84.4 (DIN)
- new net: D80.2 (DOUT), D81.4 (DIN)
- new net: D79.2 (DOUT), D80.4 (DIN)
- new net: D84.2 (DOUT), D85.4 (DIN)
- new net: D85.2 (DOUT), D86.4 (DIN)
- new net: D86.2 (DOUT), D87.4 (DIN)
- new net: D87.2 (DOUT), D88.4 (DIN)
- new net: D88.2 (DOUT), D92.4 (DIN)
- new net: D94.2 (DOUT), D98.4 (DIN)
- new net: D93.2 (DOUT), D94.4 (DIN)
- new net: D92.2 (DOUT), D93.4 (DIN)
- new net: D98.2 (DOUT), D99.4 (DIN)
- new net: D89.2 (DOUT), D90.4 (DIN)
- new net: D90.2 (DOUT), D91.4 (DIN)
- new net: D91.2 (DOUT), D95.4 (DIN)
- new net: D100.4 (DIN), D97.2 (DOUT)
- new net: D96.2 (DOUT), D97.4 (DIN)
- new net: D95.2 (DOUT), D96.4 (DIN)
- new net: D100.2 (DOUT), D101.4 (DIN)
- new net Col0: SW1.1, SW2.1, SW3.1, SW4.1, SW5.1
- new net Col1: SW10.1, SW6.1, SW7.1, SW8.1, SW9.1
- new net Col10: SW47.1, SW48.1, SW49.1, SW50.1, SW51.1
- new net Col11: SW52.1, SW53.1, SW54.1, SW55.1, SW56.1
- new net Col12: SW57.1, SW58.1, SW59.1, SW60.1, SW61.1
- new net Col13: SW62.A, SW63.A, SW64.A, SW65.A
- new net Col14: SW62.B, SW63.B, SW64.B, SW65.B
- new net Col15: SW62.S1, SW63.S1, SW64.S1, SW65.S1
- new net Col2: SW11.1, SW12.1, SW13.1, SW14.1, SW15.1
- new net Col3: SW16.1, SW17.1, SW18.1, SW19.1
- new net Col4: SW20.1, SW21.1, SW22.1, SW23.1
- new net Col5: SW24.1, SW25.1, SW26.1, SW27.1, SW28.1
- new net Col6: SW29.1, SW30.1, SW31.1, SW32.1
- new net Col7: SW33.1, SW34.1, SW35.1, SW36.1
- new net Col8: SW37.1, SW38.1, SW39.1, SW40.1, SW41.1
- new net Col9: SW42.1, SW43.1, SW44.1, SW45.1, SW46.1
- new net GND: U1.22 (GND), U1.53 (GND), U1.63 (GND)
- new net Row0: D1.1 (K), D11.1 (K), D16.1 (K), D20.1 (K), D24.1 (K), D29.1 (K), D33.1 (K), D37.1 (K), D42.1 (K), D47.1 (K), D52.1 (K), D57.1 (K), D6.1 (K), D62.1 (K), D66.1 (K)
- new net Row1: D12.1 (K), D17.1 (K), D2.1 (K), D21.1 (K), D25.1 (K), D30.1 (K), D34.1 (K), D38.1 (K), D43.1 (K), D48.1 (K), D53.1 (K), D58.1 (K), D63.1 (K), D67.1 (K), D7.1 (K)
- new net Row2: D13.1 (K), D18.1 (K), D22.1 (K), D26.1 (K), D3.1 (K), D31.1 (K), D35.1 (K), D39.1 (K), D44.1 (K), D49.1 (K), D54.1 (K), D59.1 (K), D64.1 (K), D68.1 (K), D8.1 (K)
- new net Row3: D14.1 (K), D19.1 (K), D23.1 (K), D27.1 (K), D32.1 (K), D36.1 (K), D4.1 (K), D40.1 (K), D45.1 (K), D50.1 (K), D55.1 (K), D60.1 (K), D65.1 (K), D69.1 (K), D9.1 (K)
- new net Row4: D10.1 (K), D15.1 (K), D28.1 (K), D41.1 (K), D46.1 (K), D5.1 (K), D51.1 (K), D56.1 (K), D61.1 (K)
- new net encoders: D70.4 (DIN)
Other:
- moved on the sheet: C1, C2, X1
